Commit message: tb3_custom: Migrate IMU to tinkerforge_imu2

File: turtlebot3_description/urdf/turtlebot3_custom.urdf.xacro (robot description, xacro)
@@ -34,5 +34,5 @@
     <parent link="base_link"/>
     <child link="wheel_left_link"/>
-    <origin xyz="0.0 0.08 0.023" rpy="${-M_PI*0.5} 0 0"/>
+    <origin xyz="0.0 0.0865 0.023" rpy="${-M_PI*0.5} 0 0"/>
     <axis xyz="0 0 1"/>
   </joint>
@@ -62,5 +62,5 @@
     <parent link="base_link"/>
     <child link="wheel_right_link"/>
-    <origin xyz="0.0 -0.08 0.023" rpy="${-M_PI*0.5} 0 0"/>
+    <origin xyz="0.0 -0.0865 0.023" rpy="${-M_PI*0.5} 0 0"/>
     <axis xyz="0 0 1"/>
   </joint>
@@ -108,10 +108,10 @@
   </link>
   <!-- TurtleBot3 Sensors-->
-<!--  <joint name="imu_joint" type="fixed">
+  <joint name="imu_joint" type="fixed">
     <parent link="base_link"/>
-    <child link="imu_link"/>
+    <child link="base_imu_link"/>
     <origin xyz="0.0 0 0.058" rpy="0 0 0"/>
   </joint>
-  <link name="imu_link">
+  <link name="base_imu_link">
     <inertial>
       <origin xyz="0 0 0" />
@@ -121,9 +121,9 @@
                izz="0.001" />
     </inertial>
-  </link>-->
+  </link>
   <joint name="scan_joint" type="fixed">
     <parent link="base_link"/>
     <child link="base_scan"/>
-    <origin xyz="-0.032 0 0.171" rpy="0 0 0"/>
+    <origin xyz="-0.03 0 0.171" rpy="0 0 0"/>
   </joint>
   <link name="base_scan">
